Commit message: Added rviz.launch to atlas_legs_plain, atlas_plain, atlas_plain_pinned, dreamer, dreamer_hand, dreamer_testbed, stickbot_humanoid_32dof_pinned.

File: atlas_legs_plain/models/atlas_legs_plain/xacro/atlas_legs_plain_linked_to_world.xacro (robot description, xacro)
@@ -13,5 +13,5 @@
     </link>
     <joint name="pelvisOffset" type="fixed">
-        <origin rpy="0 0 0" xyz="0 0 0"/>
+        <origin rpy="0 0 0" xyz="0 0 0.925"/>
         <axis xyz="0 0 1"/>
         <parent link="world"/>

File: atlas_plain/models/atlas_plain/xacro/atlas_plain_with_sandia_hands_linked_to_world.xacro (robot description, xacro)
@@ -12,5 +12,5 @@
     </link>
     <joint name="pelvisOffset" type="fixed">
-        <origin rpy="0 0 0" xyz="0 0 0"/>
+        <origin rpy="0 0 0" xyz="0 0 0.925"/>
         <axis xyz="0 0 1"/>
         <parent link="world"/>

File: dreamer/models/dreamer/xacro/dreamer_base.xacro (robot description, xacro)
@@ -12,5 +12,5 @@
     <property name="MESH_EXTENSION" value="stl" />
     <property name="MESH_COLL" value="low_res" />
-    <xacro:include filename="$(find hcrl_simulator)/models/generic_models.xml" />
+    <xacro:include filename="$(find controlit_models_common)/models/generic_models.xml" />
     <!--Torso-->
     <xacro:include filename="$(find dreamer)/models/dreamer/xacro/dreamer_torso.xacro"/>
@@ -60,5 +60,5 @@
     -->
     <!-- Torso joints -->
-    <gazebo reference="torso_yaw">
+    <!-- <gazebo reference="torso_yaw">
       <provideFeedback value="true"/>
     </gazebo>
@@ -68,7 +68,7 @@
     <gazebo reference="torso_upper_pitch">
       <provideFeedback value="true"/>
-    </gazebo>
+    </gazebo> -->
     <!-- right arm joints -->
-    <gazebo reference="right_shoulder_extensor">
+    <!-- <gazebo reference="right_shoulder_extensor">
       <provideFeedback value="true"/>
     </gazebo>
@@ -90,7 +90,7 @@
     <gazebo reference="right_wrist_yaw">
       <provideFeedback value="true"/>
-    </gazebo>
+    </gazebo> -->
     <!-- Left arm joints -->
-    <gazebo reference="left_shoulder_extensor">
+    <!-- <gazebo reference="left_shoulder_extensor">
       <provideFeedback value="true"/>
     </gazebo>
@@ -112,7 +112,7 @@
     <gazebo reference="left_wrist_yaw">
       <provideFeedback value="true"/>
-    </gazebo>
+    </gazebo> -->
     <!-- Head and neck joints -->
-    <gazebo reference="lower_neck_pitch">
+    <!-- <gazebo reference="lower_neck_pitch">
       <provideFeedback value="true"/>
     </gazebo>
@@ -134,7 +134,7 @@
     <gazebo reference="left_eye_yaw">
       <provideFeedback value="true"/>
-    </gazebo>
+    </gazebo> -->
     <!-- Right hand joints -->
-    <gazebo reference="right_thumb_1">
+    <!-- <gazebo reference="right_thumb_1">
       <provideFeedback value="true"/>
     </gazebo>
@@ -171,7 +171,7 @@
     <gazebo reference="right_pinky_3">
       <provideFeedback value="true"/>
-    </gazebo>
+    </gazebo> -->
     <!-- Left gripper joints -->
-    <gazebo reference="l_gripper_l_finger_joint">
+    <!-- <gazebo reference="l_gripper_l_finger_joint">
       <provideFeedback value="true"/>
     </gazebo>
@@ -184,4 +184,4 @@
     <gazebo reference="l_gripper_r_finger_tip_joint">
       <provideFeedback value="true"/>
-    </gazebo>
+    </gazebo> -->
 </robot>

File: dreamer_hand/models/dreamer_hand/xacro/dreamer_hand.xacro (robot description, xacro)
@@ -4,14 +4,7 @@
   <!-- <property name="HAND_JOINT_TYPE" value="revolute" /> -->
   <!-- For debugging purposes, fix the hand joints -->
-  <property name="HAND_JOINT_TYPE" value="revolute" />
+  <property name="RIGHT_HAND_JOINT_TYPE" value="revolute" />
   <!-- Gazebo uses model:// for the model path. -->
   <property name="modelPath" value="model://dreamer" />
   <xacro:include filename="$(find dreamer_hand)/models/dreamer_hand/xacro/dreamer_hand_base.xacro" />
-  <gazebo version='1.2'>
-      <!-- The following plugin pins the robot to the world. -->
-      <plugin filename="libPinPlugin.so" name="PinPlugin">
-          <pin_root_link>1</pin_root_link>
-      </plugin>
-      <plugin filename="libdreamer_hand_poscom_plugin.so" name="RightHandPosComPlugin"/>
-  </gazebo>
 </robot>

File: dreamer_hand/models/dreamer_hand/xacro/dreamer_hand_base.xacro (robot description, xacro)
@@ -1,27 +1,29 @@
 <?xml version="1.0"?>
 <robot xmlns:xacro="http://ros.org/wiki/xacro" name="dreamer_hand">
-  <property name="M_PI" value="3.1415926535897931" />
-  <property name="R_HAND" value="mh8" />
-  <property name="MESH" value="mid_res" />
-  <property name="MESH_COLL" value="low_res" />
-  <xacro:include filename="$(find hcrl_simulator)/models/generic_models.xml" />
-  <!-- Meka Hand -->
-  <xacro:include filename="$(find dreamer)/models/dreamer/meka_description/urdf/H2R2_r_hand_defs.urdf.xacro" />
-  <property name="M_PI" value="3.1415926535897931" />
-  <material name="GreyA"> <!-- darkest -->
-    <color rgba="0.3 0.3 0.3 1.0"/>
-  </material>
-  <material name="GreyB">
-    <color rgba="0.5 0.5 0.5 1.0"/>
-  </material>
-  <material name="GreyC">
-    <color rgba="0.7 0.7 0.7 1.0"/>
-  </material>
-  <!-- ===== DUMMY 'BASE' LINK ==== -->
-   <xacro:virtual_link name="dreamer_hand_base"
-                      origin_xyz="0 0 0.0"
-                      origin_rpy="0 0 0" />
-  <m3_r_hand side="r" reflect="1" parent="dreamer_hand_base">
-    <origin xyz="0.0 0.0 0.0" rpy="0 0 0" />
-  </m3_r_hand>
+    <property name="M_PI" value="3.1415926535897931" />
+    <property name="R_HAND" value="mh8" />
+    <property name="MESH" value="mid_res" />
+    <property name="MESH_COLL" value="low_res" />
+    <property name="MESH_QUALITY" value="optimized" />
+    <property name="RIGHT_HAND_JOINT_TYPE" value="revolute" />
+    <xacro:include filename="$(find controlit_models_common)/models/generic_models.xml" />
+    <!-- Meka Hand -->
+    <xacro:include filename="$(find dreamer)/models/dreamer/meka_description/urdf/H2R2_r_hand_defs.urdf.xacro" />
+    <property name="M_PI" value="3.1415926535897931" />
+    <material name="GreyA"> <!-- darkest -->
+        <color rgba="0.3 0.3 0.3 1.0"/>
+    </material>
+    <material name="GreyB">
+        <color rgba="0.5 0.5 0.5 1.0"/>
+    </material>
+    <material name="GreyC">
+        <color rgba="0.7 0.7 0.7 1.0"/>
+    </material>
+    <!-- ===== DUMMY 'BASE' LINK ==== -->
+     <xacro:virtual_link name="dreamer_hand_base"
+                        origin_xyz="0 0 0.0"
+                        origin_rpy="0 0 0" />
+    <m3_r_hand side="r" reflect="1" parent="dreamer_hand_base">
+        <origin xyz="0.0 0.0 0.0" rpy="0 0 0" />
+    </m3_r_hand>
 </robot>

File: dreamer_hand/models/dreamer_hand/xacro/dreamer_hand_linked_to_world.xacro (robot description, xacro)
@@ -4,5 +4,5 @@
   <!-- <property name="HAND_JOINT_TYPE" value="revolute" /> -->
   <!-- For debugging purposes, fix the hand joints -->
-  <property name="HAND_JOINT_TYPE" value="revolute" />
+  <!-- <property name="HAND_JOINT_TYPE" value="revolute" /> -->
   <!-- Gazebo uses model:// for the model path. -->
   <property name="modelPath" value="package://dreamer/models/dreamer" />
@@ -17,5 +17,5 @@
   </link>
   <joint name="baseOffset" type="fixed">
-    <origin rpy="0 0 0" xyz="0 0 0"/>
+    <origin rpy="0 0 0" xyz="0 0 0.5"/>
     <axis xyz="0 0 1"/>
     <parent link="world"/>

File: dreamer_testbed/models/dreamer_testbed/xacro/dreamer_testbed.xacro (robot description, xacro)
@@ -7,27 +7,3 @@
   <property name="modelPath" value="model://dreamer" />
   <xacro:include filename="$(find dreamer_testbed)/models/dreamer_testbed/xacro/dreamer_testbed_base.xacro" />
-  <gazebo version='1.2'>
-    <!-- The following plugin pins the robot to the world. -->
-    <plugin filename="libPinPlugin.so" name="PinPlugin">
-        <pin_root_link>1</pin_root_link>
-    </plugin>
-    <!-- The following plugin provides ground-truth odometry -->
-    <!-- <plugin filename="libgazebo_ros_p3d.so" name="pos_plugin_ros">
-      <alwaysOn>true</alwaysOn>
-      <updateRate>1000.0</updateRate>
-      <bodyName>panplate</bodyName>
-      <topicName>/dreamer_no_left_arm/pose</topicName>
-      <frameName>world</frameName>
-      <rpyOffset>0 0 0</rpyOffset>
-      <xyzOffset>0 0 1.0</xyzOffset>
-    </plugin> -->
-    <!-- The following plugin enables the hands to be controlled. -->
-    <plugin filename="libdreamer_hand_poscom_plugin.so" name="RightHandPosComPlugin"/>
-    <!-- The following plugin enables the cameras to be controlled. -->
-    <plugin filename="libdreamer_testbed_plugin.so" name="TestbedCameraControlPlugin"/>
-    <!-- The following plugin mimics the internal transmission. -->
-    <plugin filename="libdreamer_slave_joint_plugin.so" name="DreamerSlaveJointPlugin"/>
-    <!-- The following plugin controls the eyes. -->
-    <plugin filename="libdreamer_eye_plugin.so" name="DreamerEyePlugin"/>
-  </gazebo>
 </robot>

File: dreamer_testbed/models/dreamer_testbed/xacro/dreamer_testbed_base.xacro (robot description, xacro)
@@ -1,50 +1,61 @@
 <?xml version="1.0"?>
 <robot xmlns:xacro="http://playerstage.sourceforge.net/gazebo/xmlschema/#interface" name="dreamer_testbed">
-  <property name="M_PI" value="3.1415926535897931" />
-  <property name="R_ARM" value="ma10" />
-  <property name="R_HAND" value="mh8" />
-  <property name="TORSO" value="mt3" />
-  <property name="HEAD" value="ms2" />
-  <property name="MESH" value="mid_res" />
-  <property name="MESH_COLL" value="low_res" />
-  <!-- 80/20 properties-->
-  <property name="KgPerM" value="1.0715" />
-  <property name="SideLength" value="0.0381"/>
-  <property name="SideLengthSquared" value="0.00145161"/>
-  <property name="StandHeight" value="0.8"/>
-  <xacro:include filename="$(find hcrl_simulator)/models/generic_models.xml" />
-  <!--Testbed-->
-  <xacro:include filename="$(find dreamer_testbed)/models/dreamer_testbed/xacro/testbed.xacro"/>
-  <!--Torso-->
-  <xacro:include filename="$(find dreamer_no_left_arm)/models/dreamer_no_left_arm/xacro/dreamer_torso.xacro"/>
-  <!-- Meka Arm -->
-  <xacro:include filename="$(find dreamer)/models/dreamer/meka_description/urdf/A2R3_r_arm_defs.urdf.xacro" />
-  <!-- Meka Hand -->
-  <xacro:include filename="$(find dreamer)/models/dreamer/meka_description/urdf/H2R2_r_hand_defs.urdf.xacro" />
-  <!-- Meka Head -->
-  <xacro:include filename="$(find dreamer)/models/dreamer/meka_description/urdf/S2R1_head_defs.urdf.xacro" />
-  <property name="M_PI" value="3.1415926535897931" />
-  <material name="GreyA"> <!-- darkest -->
-    <color rgba="0.3 0.3 0.3 1.0"/>
-  </material>
-  <material name="GreyB">
-    <color rgba="0.5 0.5 0.5 1.0"/>
-  </material>
-  <material name="GreyC">
-    <color rgba="0.7 0.7 0.7 1.0"/>
-  </material>
-  <m3_r_arm side="r" reflect="1" parent="upper">
-    <origin xyz="0.0 -0.18465 0.2337" rpy="0 0 0" />
-  </m3_r_arm>
-  <m3_head side="r" reflect="1" parent="upper">
-    <origin xyz="0.0 0.0 0.31155" rpy="0 0 0" />
-  </m3_head>
-  <m3_r_hand side="r" reflect="1" parent="handmount_RIGHT">
-    <origin xyz="0.0 0.0 0.0" rpy="0 0 0" />
-  </m3_r_hand>
-  <testbed PARENT="panplate" stand_height="${StandHeight}" arm_back="0.25" arm_up="1.05" arm_forward="0.65" arm_drop="0.1">
-    <origin xyz="0.0 0.0 0.0" rpy="0 0 0"/>
-  </testbed>
-  <dreamer_torso height="${StandHeight}" />
+    <property name="M_PI" value="3.1415926535897931" />
+    <property name="R_ARM" value="ma10" />
+    <property name="R_HAND" value="mh8" />
+    <property name="TORSO" value="mt3" />
+    <property name="HEAD" value="ms2" />
+    <property name="MESH" value="mid_res" />
+    <property name="MESH_COLL" value="low_res" />
+    <!-- 80/20 properties-->
+    <property name="KgPerM" value="1.0715" />
+    <property name="SideLength" value="0.0381"/>
+    <property name="SideLengthSquared" value="0.00145161"/>
+    <property name="StandHeight" value="0.8"/>
+    <xacro:include filename="$(find controlit_models_common)/models/generic_models.xml" />
+    <!--Testbed-->
+    <xacro:include filename="$(find dreamer_testbed)/models/dreamer_testbed/xacro/testbed.xacro"/>
+    <!--Torso-->
+    <xacro:include filename="$(find dreamer)/models/dreamer/xacro/dreamer_torso.xacro"/>
+    <!-- Meka Right Arm -->
+    <xacro:include filename="$(find dreamer)/models/dreamer/meka_description/urdf/A2R3_r_arm_defs.urdf.xacro" />
+    <!-- Meka Left Arm -->
+    <xacro:include filename="$(find dreamer)/models/dreamer/meka_description/urdf/A2R3_l_arm_defs.urdf.xacro" />
+    <!-- Meka Hand -->
+    <xacro:include filename="$(find dreamer)/models/dreamer/meka_description/urdf/H2R2_r_hand_defs.urdf.xacro" />
+    <!-- Meka Head -->
+    <xacro:include filename="$(find dreamer)/models/dreamer/meka_description/urdf/S2R1_head_defs.urdf.xacro" />
+    <property name="M_PI" value="3.1415926535897931" />
+    <material name="GreyA"> <!-- darkest -->
+        <color rgba="0.3 0.3 0.3 1.0"/>
+    </material>
+    <material name="GreyB">
+        <color rgba="0.5 0.5 0.5 1.0"/>
+    </material>
+    <material name="GreyC">
+        <color rgba="0.7 0.7 0.7 1.0"/>
+    </material>
+    <m3_r_arm side="r" reflect="1" parent="torso_upper_pitch_link">
+        <origin xyz="0.0 -0.18465 0.2337" rpy="0 0 0" />
+    </m3_r_arm>
+    <m3_head side="r" reflect="1" parent="torso_upper_pitch_link">
+        <origin xyz="0.0 0.0 0.31155" rpy="0 0 0" />
+    </m3_head>
+    <m3_r_hand side="r" reflect="1" parent="right_wrist_yaw_link">
+        <origin xyz="0.0 0.0 0.0" rpy="0 0 0" />
+    </m3_r_hand>
+    <m3_l_arm side="l" reflect="0" parent="torso_upper_pitch_link">
+        <origin xyz="0.0 0.18465 0.2337" rpy="0 0 0" />
+    </m3_l_arm>
+    <property name="gripperModelPath" value="package://dreamer/models/dreamer" />
+    <!-- Add PR2 gripper onto end of left arm -->
+    <xacro:include filename="$(find dreamer)/models/dreamer/xacro/gripper_v0/gripper.urdf.xacro" />
+    <xacro:pr2_gripper_v0 reflect="1.0" side="l" parent="left_wrist_yaw_link" >
+        <origin xyz="0 0 0" rpy="1.57 1.57 0" />
+    </xacro:pr2_gripper_v0>
+    <testbed PARENT="panplate_link" stand_height="${StandHeight}" arm_back="0.25" arm_up="1.05" arm_forward="0.65" arm_drop="0.1">
+        <origin xyz="0.0 0.0 0.0" rpy="0 0 0"/>
+    </testbed>
+    <dreamer_torso height="${StandHeight}" />
   <!--
   The following enables torque feedback.  Without these, the following warning will be printed
@@ -52,5 +63,5 @@
   Warning [ODEJoint.cc:1105] GetForceTorque: forgot to set <provide_feedback>?
   -->
-  <gazebo reference="m3joint_mt3_j0">
+<!--   <gazebo reference="m3joint_mt3_j0">
     <provideFeedback value="true"/>
   </gazebo>
@@ -93,4 +104,4 @@
   <gazebo reference="m3joint_ms2_j3">
     <provideFeedback value="true"/>
-  </gazebo>
+  </gazebo> -->
 </robot>

File: dreamer_testbed/models/dreamer_testbed/xacro/dreamer_testbed_linked_to_world.xacro (robot description, xacro)
@@ -1,23 +1,48 @@
 <?xml version="1.0"?>
 <robot xmlns:xacro="http://ros.org/wiki/xacro" name="dreamer_testbed">
-  <!-- Gazebo should model all of the joints in the robot.  -->
-  <property name="HAND_JOINT_TYPE" value="continuous" />
-  <property name="EYE_JOINT_TYPE" value="continuous" />
-  <!-- Gazebo uses model:// for the model path. -->
-  <property name="modelPath" value="package://dreamer/models/dreamer" />
-  <xacro:include filename="$(find dreamer_testbed)/models/dreamer_testbed/xacro/dreamer_testbed_base.xacro" />
-  <link name="world">
-    <!-- Virtual Link -->
-    <inertial>
-      <mass value="0.1"/>
-      <origin rpy="0 0 0" xyz="0 0 1.2"/>
-      <inertia ixx="8.33333333333e-05" ixy="0.0" ixz="0.0" iyy="8.33333333333e-05" iyz="0.0" izz="0.000125"/>
-    </inertial>
-  </link>
-  <joint name="panplateOffset" type="fixed">
-    <origin rpy="0 0 0" xyz="0 0 0"/>
-    <axis xyz="0 0 1"/>
-    <parent link="world"/>
-    <child link="panplate"/>
-  </joint>
+    <!-- Gazebo should model all of the joints in the robot.  -->
+    <property name="HAND_JOINT_TYPE" value="continuous" />
+    <property name="EYE_JOINT_TYPE" value="continuous" />
+    <property name="RIGHT_HAND_JOINT_TYPE" value="revolute" />
+    <property name="LEFT_GRIPPER_JOINT_TYPE" value="revolute" />
+    <property name="JOINT_TYPE_TORSO_YAW"               value="fixed" />
+    <property name="JOINT_TYPE_TORSO_LOWER_PITCH"       value="revolute" />
+    <property name="JOINT_TYPE_TORSO_UPPER_PITCH"       value="revolute" />
+    <property name="JOINT_TYPE_LOWER_NECK_PITCH"        value="fixed" />
+    <property name="JOINT_TYPE_UPPER_NECK_YAW"          value="fixed" />
+    <property name="JOINT_TYPE_UPPER_NECK_ROLL"         value="fixed" />
+    <property name="JOINT_TYPE_UPPER_NECK_PITCH"        value="fixed" />
+    <property name="JOINT_TYPE_LEFT_SHOULDER_EXTENSOR"  value="revolute" />
+    <property name="JOINT_TYPE_LEFT_SHOULDER_ABDUCTOR"  value="revolute" />
+    <property name="JOINT_TYPE_LEFT_SHOULDER_ROTATOR"   value="revolute" />
+    <property name="JOINT_TYPE_LEFT_ELBOW"              value="revolute" />
+    <property name="JOINT_TYPE_LEFT_WRIST_ROTATOR"      value="revolute" />
+    <property name="JOINT_TYPE_LEFT_WRIST_PITCH"        value="revolute" />
+    <property name="JOINT_TYPE_LEFT_WRIST_YAW"          value="revolute" />
+    <property name="JOINT_TYPE_RIGHT_SHOULDER_EXTENSOR" value="revolute" />
+    <property name="JOINT_TYPE_RIGHT_SHOULDER_ABDUCTOR" value="revolute" />
+    <property name="JOINT_TYPE_RIGHT_SHOULDER_ROTATOR"  value="revolute" />
+    <property name="JOINT_TYPE_RIGHT_ELBOW"             value="revolute" />
+    <property name="JOINT_TYPE_RIGHT_WRIST_ROTATOR"     value="revolute" />
+    <property name="JOINT_TYPE_RIGHT_WRIST_PITCH"       value="revolute" />
+    <property name="JOINT_TYPE_RIGHT_WRIST_YAW"         value="revolute" />
+    <property name="MESH_QUALITY" value="optimized" />
+    <property name="MESH_EXTENSION" value="stl" />
+    <!-- Gazebo uses model:// for the model path. -->
+    <property name="modelPath" value="package://dreamer/models/dreamer" />
+    <xacro:include filename="$(find dreamer_testbed)/models/dreamer_testbed/xacro/dreamer_testbed_base.xacro" />
+    <link name="world">
+        <!-- Virtual Link -->
+        <inertial>
+            <mass value="0.1"/>
+            <origin rpy="0 0 0" xyz="0 0 1.2"/>
+            <inertia ixx="8.33333333333e-05" ixy="0.0" ixz="0.0" iyy="8.33333333333e-05" iyz="0.0" izz="0.000125"/>
+        </inertial>
+    </link>
+    <joint name="panplateOffset" type="fixed">
+        <origin rpy="0 0 0" xyz="0 0 0"/>
+        <axis xyz="0 0 1"/>
+        <parent link="world"/>
+        <child link="panplate_link"/>
+    </joint>
 </robot>
