Commit message: xacro style guide, cmake adjustments

File: atlas_legs_plain/models/atlas_legs_plain/xacro/atlas_legs_plain_base.xacro (robot description, xacro)
@@ -1,5 +1,5 @@
 <?xml version="1.0" ?>
 <robot name="atlas_legs_plain">
-    <macro name="atlas_legs_plain">
+    <xacro:macro name="atlas_legs_plain">
         <link name="l_foot">
             <inertial>
@@ -373,4 +373,4 @@
             <safety_controller k_position="100" k_velocity="100" soft_lower_limit="-10" soft_upper_limit="12.3857" />
         </joint>
-    </macro>
+    </xacro:macro>
 </robot>

File: atlas_legs_plain/models/atlas_legs_plain/xacro/atlas_legs_plain_linked_to_world.xacro (robot description, xacro)
@@ -1,5 +1,5 @@
 <robot xmlns:xacro="http://www.ros.org/wiki/xacro" name="atlas_legs_plain" >
     <!-- rViz uses package:// for the model path. -->
-    <property name="modelPath" value="package://atlas_plain/models/atlas_plain" />
+    <xacro:property name="modelPath" value="package://atlas_plain/models/atlas_plain" />
     <xacro:include filename="$(find atlas_legs_plain)/models/atlas_legs_plain/xacro/atlas_legs_plain_base.xacro" />
     <atlas_legs_plain />

File: atlas_plain/models/atlas_plain/xacro/atlas_plain_with_sandia_hands_linked_to_world.xacro (robot description, xacro)
@@ -1,5 +1,5 @@
 <robot xmlns:xacro="http://www.ros.org/wiki/xacro" name="atlas" >
     <!-- rViz uses package:// for the model path. -->
-    <property name="modelPath" value="package://atlas_plain/models/atlas_plain" />
+    <xacro:property name="modelPath" value="package://atlas_plain/models/atlas_plain" />
     <xacro:include filename="$(find atlas_plain)/models/atlas_plain/xacro/atlas_plain_with_sandia_hands.xacro" />
     <link name="world">

File: atlas_plain/models/sandia_hands/xacro/sandia_hand.urdf.xacro (robot description, xacro)
@@ -183,5 +183,5 @@
       <parent link="${parent}"/>
       <child link="${side}_palm"/>
-      <insert_block name="origin" />
+      <xacro:insert_block name="origin" />
     </joint>
     <xacro:finger side="${side}" idx="0" x="0.140" y="0.00000" z="0" r="0" p="0" yaw="0.3"/>

File: atlas_plain/models/sandia_hands/xacro/sandia_hand_simple_shapes.urdf.xacro (robot description, xacro)
@@ -405,5 +405,5 @@
       <parent link="${parent}"/>
       <child link="${side}_palm"/>
-      <insert_block name="origin" />
+      <xacro:insert_block name="origin" />
     </joint>
     <xacro:finger side="${side}" idx="0" x="0.140" y="0.00000" z="0" r="0" p="0" yaw="${0.3*reflect}" reflect="${reflect}" joint_type="${joint_type}"/>

File: dreamer/models/dreamer/meka_description/gazebo/gazebo.urdf.xacro (robot description, xacro)
@@ -1,6 +1,4 @@
 <?xml version="1.0"?>
-<robot xmlns:sensor="http://playerstage.sourceforge.net/gazebo/xmlschema/#sensor"
-       xmlns:controller="http://playerstage.sourceforge.net/gazebo/xmlschema/#controller"
-       xmlns:interface="http://playerstage.sourceforge.net/gazebo/xmlschema/#interface">
+<robot xmlns:xacro="http://ros.org/wiki/xacro">
   <gazebo>
     <controller:gazebo_ros_controller_manager name="gazebo_ros_controller_manager" plugin="libgazebo_ros_controller_manager.so">

File: dreamer/models/dreamer/meka_description/transmissions/A2R1_l_arm_defs.transmission.xacro (robot description, xacro)
@@ -1,7 +1,5 @@
 <?xml version="1.0"?>
-<robot xmlns:sensor="http://playerstage.sourceforge.net/gazebo/xmlschema/#sensor"
-       xmlns:controller="http://playerstage.sourceforge.net/gazebo/xmlschema/#controller"
-       xmlns:interface="http://playerstage.sourceforge.net/gazebo/xmlschema/#interface">
-  <macro name="m3_l_shoulder_transmission" params="side parent reflect *origin">
+<robot xmlns:xacro="http://ros.org/wiki/xacro">
+  <xacro:macro name="m3_l_shoulder_transmission" params="side parent reflect *origin">
     <!-- Shoulder pan -->
     <transmission name="m3joint_${L_ARM}_t0" type="loadable_transmissions/SimpleTransmission">
@@ -22,7 +20,7 @@
       <mechanicalReduction>1</mechanicalReduction>
     </transmission>
-  </macro>
+  </xacro:macro>
   <!-- ============================   Upper Arm   ============================ -->
-  <macro name="m3_l_upper_arm_transmission" params="side parent reflect">
+  <xacro:macro name="m3_l_upper_arm_transmission" params="side parent reflect">
     <transmission name="m3joint_${L_ARM}_t3" type="loadable_transmissions/SimpleTransmission">
       <actuator name="m3joint_${L_ARM}_a3" />
@@ -37,5 +35,5 @@
     </transmission>
   <!-- ============================   Forearm   ============================ -->
-  <macro name="m3_l_forearm_transmission" params="side parent reflect">
+  <xacro:macro name="m3_l_forearm_transmission" params="side parent reflect">
     <transmission name="m3joint_${L_ARM}_t5" type="loadable_transmissions/SimpleTransmission">
       <actuator name="m3joint_${L_ARM}_a5" />
@@ -49,9 +47,9 @@
       <mechanicalReduction>1</mechanicalReduction>
     </transmission>
-  </macro>
-  <macro name="m3_l_arm_transmission" params="side parent reflect *origin">
+  </xacro:macro>
+  <xacro:macro name="m3_l_arm_transmission" params="side parent reflect *origin">
     <m3_l_shoulde_transmissionr side="${side}" reflect="${reflect}" parent="${parent}"/>
     <m3_l_upper_ar_transmissionm side="${side}" reflect="${reflect}" parent="bicep_LEFT" />
     <m3_l_forear_transmissionm side="${side}" reflect="${reflect}" parent="wrist_LEFT" />
-  </macro>
+  </xacro:macro>
 </robot>

File: dreamer/models/dreamer/meka_description/transmissions/A2R1_r_arm_defs.transmission.xacro (robot description, xacro)
@@ -1,7 +1,5 @@
 <?xml version="1.0"?>
-<robot xmlns:sensor="http://playerstage.sourceforge.net/gazebo/xmlschema/#sensor"
-       xmlns:controller="http://playerstage.sourceforge.net/gazebo/xmlschema/#controller"
-       xmlns:interface="http://playerstage.sourceforge.net/gazebo/xmlschema/#interface">
-  <macro name="m3_r_shoulder_transmission" params="side parent reflect *origin">
+<robot xmlns:xacro="http://ros.org/wiki/xacro">
+  <xacro:macro name="m3_r_shoulder_transmission" params="side parent reflect *origin">
     <!-- Shoulder pan -->
     <transmission name="m3joint_${R_ARM}_t0" type="loadable_transmissions/SimpleTransmission">
@@ -22,7 +20,7 @@
       <mechanicalReduction>1</mechanicalReduction>
     </transmission>
-  </macro>
+  </xacro:macro>
   <!-- ============================   Upper Arm   ============================ -->
-  <macro name="m3_r_upper_arm_transmission" params="side parent reflect">
+  <xacro:macro name="m3_r_upper_arm_transmission" params="side parent reflect">
     <transmission name="m3joint_${R_ARM}_t3" type="loadable_transmissions/SimpleTransmission">
       <actuator name="m3joint_${R_ARM}_a3" />
@@ -36,7 +34,7 @@
       <mechanicalReduction>1</mechanicalReduction>
     </transmission>
-  </macro>
+  </xacro:macro>
   <!-- ============================   Forearm   ============================ -->
-  <macro name="m3_r_forearm_transmission" params="side parent reflect">
+  <xacro:macro name="m3_r_forearm_transmission" params="side parent reflect">
     <transmission name="m3joint_${R_ARM}_t5" type="loadable_transmissions/SimpleTransmission">
       <actuator name="m3joint_${R_ARM}_a5" />
@@ -50,9 +48,9 @@
       <mechanicalReduction>1</mechanicalReduction>
     </transmission>
-  </macro>
-  <macro name="m3_r_arm_transmission" params="side parent reflect *origin">
+  </xacro:macro>
+  <xacro:macro name="m3_r_arm_transmission" params="side parent reflect *origin">
     <m3_r_shoulde_transmissionr side="${side}" reflect="${reflect}" parent="${parent}"/>
     <m3_r_upper_ar_transmissionm side="${side}" reflect="${reflect}" parent="bicep_RIGHT" />
     <m3_r_forear_transmissionm side="${side}" reflect="${reflect}" parent="wrist_RIGHT" />
-  </macro>
+  </xacro:macro>
 </robot>

File: dreamer/models/dreamer/meka_description/transmissions/A2R2_l_arm_defs.transmission.xacro (robot description, xacro)
@@ -1,7 +1,5 @@
 <?xml version="1.0"?>
-<robot xmlns:sensor="http://playerstage.sourceforge.net/gazebo/xmlschema/#sensor"
-       xmlns:controller="http://playerstage.sourceforge.net/gazebo/xmlschema/#controller"
-       xmlns:interface="http://playerstage.sourceforge.net/gazebo/xmlschema/#interface">
-  <macro name="m3_l_shoulder_transmission" params="side parent reflect">
+<robot xmlns:xacro="http://ros.org/wiki/xacro">
+  <xacro:macro name="m3_l_shoulder_transmission" params="side parent reflect">
     <!-- Shoulder pan -->
     <transmission name="m3joint_${L_ARM}_t0" type="loadable_transmissions/SimpleTransmission">
@@ -22,7 +20,7 @@
       <mechanicalReduction>1</mechanicalReduction>
     </transmission>
-  </macro>
+  </xacro:macro>
   <!-- ============================   Upper Arm   ============================ -->
-  <macro name="m3_l_upper_arm_transmission" params="side parent reflect">
+  <xacro:macro name="m3_l_upper_arm_transmission" params="side parent reflect">
     <transmission name="m3joint_${L_ARM}_t3" type="loadable_transmissions/SimpleTransmission">
       <actuator name="m3joint_${L_ARM}_a3" />
@@ -36,7 +34,7 @@
       <mechanicalReduction>1</mechanicalReduction>
     </transmission>
-  </macro>
+  </xacro:macro>
   <!-- ============================   Forearm   ============================ -->
-  <macro name="m3_l_forearm_transmission" params="side parent reflect">
+  <xacro:macro name="m3_l_forearm_transmission" params="side parent reflect">
     <transmission name="m3joint_${L_ARM}_t5" type="loadable_transmissions/SimpleTransmission">
       <actuator name="m3joint_${L_ARM}_a5" />
@@ -50,9 +48,9 @@
       <mechanicalReduction>1</mechanicalReduction>
     </transmission>
-  </macro>
-  <macro name="m3_l_arm_transmission" params="side parent reflect">
+  </xacro:macro>
+  <xacro:macro name="m3_l_arm_transmission" params="side parent reflect">
     <m3_l_shoulder_transmission side="${side}" reflect="${reflect}" parent="${parent}"/>
     <m3_l_upper_arm_transmission side="${side}" reflect="${reflect}" parent="bicep_LEFT" />
     <m3_l_forearm_transmission side="${side}" reflect="${reflect}" parent="wrist_LEFT" />
-  </macro>
+  </xacro:macro>
 </robot>

File: dreamer/models/dreamer/meka_description/transmissions/A2R2_r_arm_defs.transmission.xacro (robot description, xacro)
@@ -1,7 +1,5 @@
 <?xml version="1.0"?>
-<robot xmlns:sensor="http://playerstage.sourceforge.net/gazebo/xmlschema/#sensor"
-       xmlns:controller="http://playerstage.sourceforge.net/gazebo/xmlschema/#controller"
-       xmlns:interface="http://playerstage.sourceforge.net/gazebo/xmlschema/#interface">
-  <macro name="m3_r_shoulder_transmission" params="side parent reflect">
+<robot xmlns:xacro="http://ros.org/wiki/xacro">
+  <xacro:macro name="m3_r_shoulder_transmission" params="side parent reflect">
     <!-- Shoulder pan -->
     <transmission name="m3joint_${R_ARM}_t0" type="loadable_transmissions/SimpleTransmission">
@@ -22,7 +20,7 @@
       <mechanicalReduction>1</mechanicalReduction>
     </transmission>
-  </macro>
+  </xacro:macro>
   <!-- ============================   Upper Arm   ============================ -->
-  <macro name="m3_r_upper_arm_transmission" params="side parent reflect">
+  <xacro:macro name="m3_r_upper_arm_transmission" params="side parent reflect">
     <transmission name="m3joint_${R_ARM}_t3" type="loadable_transmissions/SimpleTransmission">
       <actuator name="m3joint_${R_ARM}_a3" />
@@ -36,7 +34,7 @@
       <mechanicalReduction>1</mechanicalReduction>
     </transmission>
-  </macro>
+  </xacro:macro>
   <!-- ============================   Forearm   ============================ -->
-  <macro name="m3_r_forearm_transmission" params="side parent reflect">
+  <xacro:macro name="m3_r_forearm_transmission" params="side parent reflect">
     <transmission name="m3joint_${R_ARM}_t5" type="loadable_transmissions/SimpleTransmission">
       <actuator name="m3joint_${R_ARM}_a5" />
@@ -50,9 +48,9 @@
       <mechanicalReduction>1</mechanicalReduction>
     </transmission>
-  </macro>
-  <macro name="m3_r_arm_transmission" params="side parent reflect">
+  </xacro:macro>
+  <xacro:macro name="m3_r_arm_transmission" params="side parent reflect">
     <m3_r_shoulder_transmission side="${side}" reflect="${reflect}" parent="${parent}"/>
     <m3_r_upper_arm_transmission side="${side}" reflect="${reflect}" parent="bicep_RIGHT" />
     <m3_r_forearm_transmission side="${side}" reflect="${reflect}" parent="wrist_RIGHT" />
-  </macro>
+  </xacro:macro>
 </robot>

File: dreamer/models/dreamer/meka_description/transmissions/A2R3_l_arm_defs.transmission.xacro (robot description, xacro)
@@ -1,7 +1,5 @@
 <?xml version="1.0"?>
-<robot xmlns:sensor="http://playerstage.sourceforge.net/gazebo/xmlschema/#sensor"
-       xmlns:controller="http://playerstage.sourceforge.net/gazebo/xmlschema/#controller"
-       xmlns:interface="http://playerstage.sourceforge.net/gazebo/xmlschema/#interface">
-  <macro name="m3_l_shoulder_transmission" params="side parent reflect *origin">
+<robot xmlns:xacro="http://ros.org/wiki/xacro">
+  <xacro:macro name="m3_l_shoulder_transmission" params="side parent reflect *origin">
     <!-- Shoulder pan -->
     <transmission name="m3joint_${L_ARM}_t0" type="loadable_transmissions/SimpleTransmission">
@@ -22,7 +20,7 @@
       <mechanicalReduction>1</mechanicalReduction>
     </transmission>
-  </macro>
+  </xacro:macro>
   <!-- ============================   Upper Arm   ============================ -->
-  <macro name="m3_l_upper_arm_transmission" params="side parent reflect">
+  <xacro:macro name="m3_l_upper_arm_transmission" params="side parent reflect">
     <transmission name="m3joint_${L_ARM}_t3" type="loadable_transmissions/SimpleTransmission">
       <actuator name="m3joint_${L_ARM}_a3" />
@@ -36,7 +34,7 @@
       <mechanicalReduction>1</mechanicalReduction>
     </transmission>
-  </macro>
+  </xacro:macro>
   <!-- ============================   Forearm   ============================ -->
-  <macro name="m3_l_forearm_transmission" params="side parent reflect">
+  <xacro:macro name="m3_l_forearm_transmission" params="side parent reflect">
     <transmission name="m3joint_${L_ARM}_t5" type="loadable_transmissions/SimpleTransmission">
       <actuator name="m3joint_${L_ARM}_a5" />
@@ -50,9 +48,9 @@
       <mechanicalReduction>1</mechanicalReduction>
     </transmission>
-  </macro>
-  <macro name="m3_l_arm_transmission" params="side parent reflect *origin">
+  </xacro:macro>
+  <xacro:macro name="m3_l_arm_transmission" params="side parent reflect *origin">
     <m3_l_shoulde_transmissionr side="${side}" reflect="${reflect}" parent="${parent}"/>
     <m3_l_upper_ar_transmissionm side="${side}" reflect="${reflect}" parent="bicep_LEFT" />
     <m3_l_forear_transmissionm side="${side}" reflect="${reflect}" parent="wrist_LEFT" />
-  </macro>
+  </xacro:macro>
 </robot>

File: dreamer/models/dreamer/meka_description/transmissions/H2R2_r_hand_defs.transmission.xacro (robot description, xacro)
@@ -1,8 +1,6 @@
 <?xml version="1.0"?>
-<robot xmlns:sensor="http://playerstage.sourceforge.net/gazebo/xmlschema/#sensor"
-       xmlns:controller="http://playerstage.sourceforge.net/gazebo/xmlschema/#controller"
-       xmlns:interface="http://playerstage.sourceforge.net/gazebo/xmlschema/#interface">
-  <property name="M_PI" value="3.1415926535897931" />
-  <macro name="m3_r_palm_transmission">
+<robot xmlns:xacro="http://ros.org/wiki/xacro">
+  <xacro:property name="M_PI" value="3.1415926535897931" />
+  <xacro:macro name="m3_r_palm_transmission">
 <!-- Start Thumb -->
   <transmission name="m3joint_ua_${R_HAND}_t0" type="loadable_transmissions/SimpleTransmission">
@@ -69,7 +67,7 @@
     <mechanicalReduction>1</mechanicalReduction>
   </transmission>
-</macro>
-  <macro name="m3_r_hand_transmission">
+</xacro:macro>
+  <xacro:macro name="m3_r_hand_transmission">
     <m3_r_palm_transmission/>
-  </macro>
+  </xacro:macro>
 </robot>

File: dreamer/models/dreamer/meka_description/transmissions/S2R1_head_defs.transmission.xacro (robot description, xacro)
@@ -1,8 +1,6 @@
 <?xml version="1.0"?>
-<robot xmlns:sensor="http://playerstage.sourceforge.net/gazebo/xmlschema/#sensor"
-       xmlns:controller="http://playerstage.sourceforge.net/gazebo/xmlschema/#controller"
-       xmlns:interface="http://playerstage.sourceforge.net/gazebo/xmlschema/#interface">
-  <property name="M_PI" value="3.1415926535897931" />
-  <macro name="m3_neck_transmission">
+<robot xmlns:xacro="http://ros.org/wiki/xacro">
+  <xacro:property name="M_PI" value="3.1415926535897931" />
+  <xacro:macro name="m3_neck_transmission">
   <transmission name="m3joint_${HEAD}_t0" type="loadable_transmissions/SimpleTransmission">
       <actuator name="m3joint_${HEAD}_a0"/>
@@ -40,7 +38,7 @@
     <mechanicalReduction>1</mechanicalReduction>
   </transmission>
-</macro>
-  <macro name="m3_head_transmission">
+</xacro:macro>
+  <xacro:macro name="m3_head_transmission">
     <m3_neck_transmission/>
-  </macro>
+  </xacro:macro>
 </robot>

File: dreamer/models/dreamer/meka_description/transmissions/m3.transmission.xacro (robot description, xacro)
@@ -1,6 +1,4 @@
 <?xml version="1.0"?>
-<robot xmlns:sensor="http://playerstage.sourceforge.net/gazebo/xmlschema/#sensor"
-       xmlns:controller="http://playerstage.sourceforge.net/gazebo/xmlschema/#controller"
-       xmlns:interface="http://playerstage.sourceforge.net/gazebo/xmlschema/#interface"
+<robot xmlns:xacro="http://ros.org/wiki/xacro"
        xmlns:xacro="http://playerstage.sourceforge.net/gazebo/xmlschema/#interface"
        name="m3" >

File: dreamer/models/dreamer/meka_description/urdf/A2R3_l_arm_defs.urdf.xacro (robot description, xacro)
@@ -1,34 +1,32 @@
 <?xml version="1.0"?>
-<robot xmlns:sensor="http://playerstage.sourceforge.net/gazebo/xmlschema/#sensor"
-       xmlns:controller="http://playerstage.sourceforge.net/gazebo/xmlschema/#controller"
-       xmlns:interface="http://playerstage.sourceforge.net/gazebo/xmlschema/#interface">
-    <property name="M_PI" value="3.1415926535897931" />
-    <property name="VELOCITY_LIMIT_SCALE" value="0.6" />
-    <property name="shoulder_lift_length" value="0.10" />
-    <property name="shoulder_lift_radius" value="0.12" />
+<robot xmlns:xacro="http://ros.org/wiki/xacro">
+    <xacro:property name="M_PI" value="3.1415926535897931" />
+    <xacro:property name="VELOCITY_LIMIT_SCALE" value="0.6" />
+    <xacro:property name="shoulder_lift_length" value="0.10" />
+    <xacro:property name="shoulder_lift_radius" value="0.12" />
     <!-- for non-symmetric upper arm -->
-    <property name="uar_xyz1" value= "0.21398" />
-    <property name="uar_xyz2" value="-0.01621" />
-    <property name="uar_xyz3" value="-0.00020" />
-    <property name="uar_ixx"  value= "0.01537748957" />
-    <property name="uar_ixy"  value= "0.00375711247" />
-    <property name="uar_ixz"  value="-0.00070852914" />
-    <property name="uar_iyy"  value= "0.07473670440" />
-    <property name="uar_iyz"  value="-0.00017936450" />
-    <property name="uar_izz"  value= "0.07608763307" />
-    <property name="ual_xyz1" value= "0.21405" />
-    <property name="ual_xyz2" value= "0.01658" />
-    <property name="ual_xyz3" value="-0.00057" />
-    <property name="ual_ixx"  value= "0.01530603856" />
-    <property name="ual_ixy"  value="-0.00339324862" />
-    <property name="ual_ixz"  value= "0.00060765455" />
-    <property name="ual_iyy"  value= "0.07473694455" />
-    <property name="ual_iyz"  value="-0.00019953729" />
-    <property name="ual_izz"  value= "0.07601594191" />
-    <macro name="m3_l_shoulder" params="side parent reflect *origin">
+    <xacro:property name="uar_xyz1" value= "0.21398" />
+    <xacro:property name="uar_xyz2" value="-0.01621" />
+    <xacro:property name="uar_xyz3" value="-0.00020" />
+    <xacro:property name="uar_ixx"  value= "0.01537748957" />
+    <xacro:property name="uar_ixy"  value= "0.00375711247" />
+    <xacro:property name="uar_ixz"  value="-0.00070852914" />
+    <xacro:property name="uar_iyy"  value= "0.07473670440" />
+    <xacro:property name="uar_iyz"  value="-0.00017936450" />
+    <xacro:property name="uar_izz"  value= "0.07608763307" />
+    <xacro:property name="ual_xyz1" value= "0.21405" />
+    <xacro:property name="ual_xyz2" value= "0.01658" />
+    <xacro:property name="ual_xyz3" value="-0.00057" />
+    <xacro:property name="ual_ixx"  value= "0.01530603856" />
+    <xacro:property name="ual_ixy"  value="-0.00339324862" />
+    <xacro:property name="ual_ixz"  value= "0.00060765455" />
+    <xacro:property name="ual_iyy"  value= "0.07473694455" />
+    <xacro:property name="ual_iyz"  value="-0.00019953729" />
+    <xacro:property name="ual_izz"  value= "0.07601594191" />
+    <xacro:macro name="m3_l_shoulder" params="side parent reflect *origin">
         <!-- Shoulder pan -->
         <joint name="left_shoulder_extensor" type="${JOINT_TYPE_LEFT_SHOULDER_EXTENSOR}">
             <axis xyz="0 -1 0" />
-            <insert_block name="origin" /> <!-- transform from parent link to this joint frame -->
+            <xacro:insert_block name="origin" /> <!-- transform from parent link to this joint frame -->
             <parent link="${parent}"/>
             <child link="left_shoulder_extensor_link"/>
@@ -127,7 +125,7 @@
             </collision>
         </link>
-    </macro>
+    </xacro:macro>
     <!-- ============================   Upper Arm   ============================ -->
-    <macro name="m3_l_upper_arm" params="side parent reflect">
+    <xacro:macro name="m3_l_upper_arm" params="side parent reflect">
         <joint name="left_elbow" type="${JOINT_TYPE_LEFT_ELBOW}">
             <axis xyz="0 1 0" />
@@ -196,7 +194,7 @@
             </collision>
         </link>
-    </macro>
+    </xacro:macro>
     <!-- ============================   Forearm   ============================ -->
-    <macro name="m3_l_forearm" params="side parent reflect">
+    <xacro:macro name="m3_l_forearm" params="side parent reflect">
         <joint name="left_wrist_pitch" type="${JOINT_TYPE_LEFT_WRIST_PITCH}">
             <dynamics damping="1.0" />
@@ -259,11 +257,11 @@
             </collision>
         </link>
-    </macro>
-    <macro name="m3_l_arm" params="side parent reflect *origin">
+    </xacro:macro>
+    <xacro:macro name="m3_l_arm" params="side parent reflect *origin">
         <m3_l_shoulder side="${side}" reflect="${reflect}" parent="${parent}">
-            <insert_block name="origin" />
+            <xacro:insert_block name="origin" />
         </m3_l_shoulder>
         <m3_l_upper_arm side="${side}" reflect="${reflect}" parent="left_shoulder_rotator_link"/>
         <m3_l_forearm side="${side}" reflect="${reflect}" parent="left_wrist_rotator_link" />
-    </macro>
+    </xacro:macro>
 </robot>
