Commit message: xacro style guide, cmake adjustments

File: dreamer/models/dreamer/meka_description/urdf/A2R3_r_arm_defs.urdf.xacro (robot description, xacro)
@@ -1,12 +1,10 @@
 <?xml version="1.0"?>
-<robot xmlns:sensor="http://playerstage.sourceforge.net/gazebo/xmlschema/#sensor"
-       xmlns:controller="http://playerstage.sourceforge.net/gazebo/xmlschema/#controller"
-       xmlns:interface="http://playerstage.sourceforge.net/gazebo/xmlschema/#interface">
-    <property name="M_PI" value="3.1415926535897931" />
-    <macro name="m3_r_shoulder" params="side parent reflect *origin">
+<robot xmlns:xacro="http://ros.org/wiki/xacro">
+    <xacro:property name="M_PI" value="3.1415926535897931" />
+    <xacro:macro name="m3_r_shoulder" params="side parent reflect *origin">
     <!-- Shoulder pan -->
     <joint name="right_shoulder_extensor" type="${JOINT_TYPE_RIGHT_SHOULDER_EXTENSOR}">
         <axis xyz="0 -1 0" />
-        <insert_block name="origin" /> <!-- transform from parent link to this joint frame -->
+        <xacro:insert_block name="origin" /> <!-- transform from parent link to this joint frame -->
         <parent link="${parent}"/>
         <child link="right_shoulder_extensor_link"/>
@@ -106,7 +104,7 @@
         </collision>
     </link>
-</macro>
+</xacro:macro>
 <!-- ============================   Upper Arm   ============================ -->
-<macro name="m3_r_upper_arm" params="side parent reflect">
+<xacro:macro name="m3_r_upper_arm" params="side parent reflect">
     <joint name="right_elbow" type="${JOINT_TYPE_RIGHT_ELBOW}">
         <axis xyz="0 -1 0" />
@@ -176,7 +174,7 @@
         </collision>
     </link>
-  </macro>
+  </xacro:macro>
   <!-- ============================   Forearm   ============================ -->
-    <macro name="m3_r_forearm" params="side parent reflect">
+    <xacro:macro name="m3_r_forearm" params="side parent reflect">
         <joint name="right_wrist_pitch" type="${JOINT_TYPE_RIGHT_WRIST_PITCH}">
             <dynamics damping="1.0" />
@@ -239,11 +237,11 @@
             </collision>
         </link>
-   </macro>
-  <macro name="m3_r_arm" params="side parent reflect *origin">
+   </xacro:macro>
+  <xacro:macro name="m3_r_arm" params="side parent reflect *origin">
     <m3_r_shoulder side="${side}" reflect="${reflect}" parent="${parent}">
-      <insert_block name="origin" />
+      <xacro:insert_block name="origin" />
     </m3_r_shoulder>
     <m3_r_upper_arm side="${side}" reflect="${reflect}" parent="right_shoulder_rotator_link" />
     <m3_r_forearm side="${side}" reflect="${reflect}" parent="right_wrist_rotator_link" />
-  </macro>
+  </xacro:macro>
 </robot>

File: dreamer/models/dreamer/meka_description/urdf/H2R2_l_hand_defs.urdf.xacro (robot description, xacro)
@@ -1,9 +1,7 @@
 <?xml version="1.0"?>
-<robot xmlns:sensor="http://playerstage.sourceforge.net/gazebo/xmlschema/#sensor"
-       xmlns:controller="http://playerstage.sourceforge.net/gazebo/xmlschema/#controller"
-       xmlns:interface="http://playerstage.sourceforge.net/gazebo/xmlschema/#interface">
-    <property name="M_PI" value="3.1415926535897931" />
+<robot xmlns:xacro="http://ros.org/wiki/xacro">
+    <xacro:property name="M_PI" value="3.1415926535897931" />
   <!-- INERTIA MATRIX CHANGE BY POLAM, VALUE=0.0011100-->
-    <macro name="m3_l_palm" params="side parent reflect *origin">
+    <xacro:macro name="m3_l_palm" params="side parent reflect *origin">
         <joint name="l_palm_joint" type="fixed">
             <origin xyz="0 0.0 -0.04414" rpy="0 0 0" />
@@ -421,9 +419,9 @@
             </collision>
         </link>
-    </macro>
-    <macro name="m3_l_hand" params="side parent reflect *origin">
+    </xacro:macro>
+    <xacro:macro name="m3_l_hand" params="side parent reflect *origin">
         <m3_l_palm side="${side}" reflect="${reflect}" parent="${parent}">
-            <insert_block name="origin" />
+            <xacro:insert_block name="origin" />
         </m3_l_palm>
-    </macro>
+    </xacro:macro>
 </robot>

File: dreamer/models/dreamer/meka_description/urdf/H2R2_r_hand_defs.urdf.xacro (robot description, xacro)
@@ -1,5 +1,5 @@
 <?xml version="1.0"?>
 <robot xmlns:xacro="http://ros.org/wiki/xacro" name="dreamer">
-    <property name="M_PI" value="3.1415926535897931" />
+    <xacro:property name="M_PI" value="3.1415926535897931" />
     <!-- INERTIA MATRIX CHANGE BY POLAM, VALUE=0.0011100-->
     <xacro:macro name="m3_r_palm" params="side parent reflect *origin">
@@ -461,5 +461,5 @@
     <xacro:macro name="m3_r_hand" params="side parent reflect *origin">
         <m3_r_palm side="${side}" reflect="${reflect}" parent="${parent}">
-            <insert_block name="origin" />
+            <xacro:insert_block name="origin" />
         </m3_r_palm>
     </xacro:macro>

File: dreamer/models/dreamer/meka_description/urdf/S2R1_head_defs.urdf.xacro (robot description, xacro)
@@ -1,12 +1,10 @@
 <?xml version="1.0"?>
-<robot xmlns:sensor="http://playerstage.sourceforge.net/gazebo/xmlschema/#sensor"
-       xmlns:controller="http://playerstage.sourceforge.net/gazebo/xmlschema/#controller"
-       xmlns:interface="http://playerstage.sourceforge.net/gazebo/xmlschema/#interface">
-    <property name="M_PI" value="3.1415926535897931" />
+<robot xmlns:xacro="http://ros.org/wiki/xacro">
+    <xacro:property name="M_PI" value="3.1415926535897931" />
     <!-- INERTIA MATRIX CHANGE BY POLAM, VALUE=0.0011100-->
-    <macro name="m3_neck" params="side parent reflect *origin">
+    <xacro:macro name="m3_neck" params="side parent reflect *origin">
         <joint name="lower_neck_pitch" type="${JOINT_TYPE_LOWER_NECK_PITCH}">
             <axis xyz="0 -1 0" />
-            <insert_block name="origin" /> <!-- transform from parent link to this joint frame -->
+            <xacro:insert_block name="origin" /> <!-- transform from parent link to this joint frame -->
             <parent link="${parent}"/>
             <child link="lower_neck_pitch_link"/>
@@ -233,9 +231,9 @@
             </collision>
         </link>
-    </macro>
-    <macro name="m3_head" params="side parent reflect *origin">
+    </xacro:macro>
+    <xacro:macro name="m3_head" params="side parent reflect *origin">
         <m3_neck side="${side}" reflect="${reflect}" parent="${parent}">
-            <insert_block name="origin" />
+            <xacro:insert_block name="origin" />
         </m3_neck>
-    </macro>
+    </xacro:macro>
 </robot>

File: dreamer/models/dreamer/xacro/dreamer_base.xacro (robot description, xacro)
@@ -1,15 +1,15 @@
 <?xml version="1.0"?>
 <robot xmlns:xacro="http://ros.org/wiki/xacro" name="dreamer">
-    <property name="M_PI" value="3.1415926535897931" />
-    <property name="R_ARM" value="ma10" />
-    <property name="L_ARM" value="l_arm" />
-    <property name="R_HAND" value="mh8" />
-    <property name="L_HAND" value="left_hand" />
-    <property name="TORSO" value="mt3" />
-    <property name="HEAD" value="ms2" />
-    <!-- <property name="MESH" value="mid_res" /> -->
-    <property name="MESH_QUALITY" value="optimized" />
-    <property name="MESH_EXTENSION" value="stl" />
-    <property name="MESH_COLL" value="low_res" />
+    <xacro:property name="M_PI" value="3.1415926535897931" />
+    <xacro:property name="R_ARM" value="ma10" />
+    <xacro:property name="L_ARM" value="l_arm" />
+    <xacro:property name="R_HAND" value="mh8" />
+    <xacro:property name="L_HAND" value="left_hand" />
+    <xacro:property name="TORSO" value="mt3" />
+    <xacro:property name="HEAD" value="ms2" />
+    <!-- <xacro:property name="MESH" value="mid_res" /> -->
+    <xacro:property name="MESH_QUALITY" value="optimized" />
+    <xacro:property name="MESH_EXTENSION" value="stl" />
+    <xacro:property name="MESH_COLL" value="low_res" />
     <xacro:include filename="$(find controlit_models_common)/models/generic_models.xml" />
     <!--Torso-->
