Commit message: Decreased mass of stickbot_humanoid_32dof to make it easier to control in simulation.

File: stickbot_humanoid_32dof/models/stickbot_humanoid_32dof/xacro/stickbot_humanoid_32dof_base.xacro (robot description, xacro)
@@ -5,5 +5,5 @@
     <link name="pelvis">
       <inertial>
-        <mass value="3"/>
+        <mass value="2"/>
         <origin xyz="0.0 0.0 0.05"/>
         <inertia ixx="0.008667" ixy="0" ixz="0" iyy="0.008667" iyz="0" izz="0.01667"/>
@@ -37,5 +37,5 @@
     <link name="leftHipLink1">
       <inertial>
-        <mass value="3.0"/>
+        <mass value="2.0"/>
         <origin xyz="0.0 0.0 -0.015"/>
         <inertia ixx="0.00015" ixy="0" ixz="0" iyy="0.00015" iyz="0" izz="0.000225"/>
@@ -68,5 +68,5 @@
     <link name="leftHipExtensorLink">
       <inertial>
-        <mass value="3.0"/>
+        <mass value="2.0"/>
         <origin xyz="0.0 0.0 -0.015"/>
         <inertia ixx="0.00015" ixy="0" ixz="0" iyy="0.00015" iyz="0" izz="0.000225"/>
@@ -224,5 +224,5 @@
     <link name="rightHipLink1">
       <inertial>
-        <mass value="3.0"/>
+        <mass value="2.0"/>
         <origin xyz="0.0 0.0 -0.015"/>
         <inertia ixx="0.00015" ixy="0" ixz="0" iyy="0.00015" iyz="0" izz="0.000225"/>
@@ -255,5 +255,5 @@
     <link name="rightHipExtensorLink">
       <inertial>
-        <mass value="3.0"/>
+        <mass value="2.0"/>
         <origin xyz="0.0 0.0 -0.015"/>
         <inertia ixx="0.00015" ixy="0" ixz="0" iyy="0.00015" iyz="0" izz="0.000225"/>
@@ -410,5 +410,5 @@
     <link name="abdomen">
       <inertial>
-        <mass value="1.5"/>
+        <mass value="1.0"/>
         <origin xyz="0.0 0.0 0.125"/>
         <inertia ixx="0.028125" ixy="0" ixz="0" iyy="0.045" iyz="0" izz="0.028125"/>
@@ -441,5 +441,5 @@
     <link name="torso">
       <inertial>
-        <mass value="3"/>
+        <mass value="2"/>
         <origin xyz="0.0 0.0 0.125"/>
         <inertia ixx="0.028125" ixy="0" ixz="0" iyy="0.045" iyz="0" izz="0.028125"/>
@@ -472,5 +472,5 @@
     <link name="chest">
       <inertial>
-        <mass value="3"/>
+        <mass value="2"/>
         <origin xyz="0.0 0.0 0.125"/>
         <inertia ixx="0.028125" ixy="0" ixz="0" iyy="0.045" iyz="0" izz="0.028125"/>
@@ -503,5 +503,5 @@
     <link name="right_shoulder_extensor">
       <inertial>
-        <mass value="3"/>
+        <mass value="1"/>
         <origin xyz="0.0 -0.01 0.0"/>
         <inertia ixx="0.028125" ixy="0" ixz="0" iyy="0.045" iyz="0" izz="0.028125"/>
@@ -534,5 +534,5 @@
     <link name="right_shoulder_adductor">
       <inertial>
-        <mass value="3"/>
+        <mass value="1"/>
         <origin xyz="0.0 -0.02 0.0"/>
         <inertia ixx="0.028125" ixy="0" ixz="0" iyy="0.045" iyz="0" izz="0.028125"/>
@@ -565,5 +565,5 @@
     <link name="right_shoulder_rotator">
       <inertial>
-        <mass value="3"/>
+        <mass value="2"/>
         <origin xyz="0.0 0.0 -0.1"/>
         <inertia ixx="0.028125" ixy="0" ixz="0" iyy="0.045" iyz="0" izz="0.028125"/>
@@ -596,5 +596,5 @@
     <link name="right_elbow_extensor">
       <inertial>
-        <mass value="3"/>
+        <mass value="2"/>
         <origin xyz="0.0 0.0 -0.1"/>
         <inertia ixx="0.028125" ixy="0" ixz="0" iyy="0.045" iyz="0" izz="0.028125"/>
@@ -627,5 +627,5 @@
     <link name="right_wrist_rotator">
       <inertial>
-        <mass value="3"/>
+        <mass value="2"/>
         <origin xyz="0.0 0.0 -0.02"/>
         <inertia ixx="0.028125" ixy="0" ixz="0" iyy="0.045" iyz="0" izz="0.028125"/>
@@ -658,5 +658,5 @@
     <link name="right_wrist_extensor">
       <inertial>
-        <mass value="3"/>
+        <mass value="1"/>
         <origin xyz="0.0 0.0 -0.02"/>
         <inertia ixx="0.028125" ixy="0" ixz="0" iyy="0.045" iyz="0" izz="0.028125"/>
@@ -689,5 +689,5 @@
     <link name="right_wrist_adductor">
       <inertial>
-        <mass value="3"/>
+        <mass value="1"/>
         <origin xyz="0.0 0.0 -0.06"/>
         <inertia ixx="0.028125" ixy="0" ixz="0" iyy="0.045" iyz="0" izz="0.028125"/>
@@ -720,5 +720,5 @@
     <link name="left_shoulder_extensor">
       <inertial>
-        <mass value="3"/>
+        <mass value="1"/>
         <origin xyz="0.0 0.01 0.0"/>
         <inertia ixx="0.028125" ixy="0" ixz="0" iyy="0.045" iyz="0" izz="0.028125"/>
@@ -751,5 +751,5 @@
     <link name="left_shoulder_adductor">
       <inertial>
-        <mass value="3"/>
+        <mass value="1"/>
         <origin xyz="0.0 0.02 0.0"/>
         <inertia ixx="0.028125" ixy="0" ixz="0" iyy="0.045" iyz="0" izz="0.028125"/>
@@ -782,5 +782,5 @@
     <link name="left_shoulder_rotator">
       <inertial>
-        <mass value="3"/>
+        <mass value="2"/>
         <origin xyz="0.0 0.0 -0.1"/>
         <inertia ixx="0.028125" ixy="0" ixz="0" iyy="0.045" iyz="0" izz="0.028125"/>
@@ -813,5 +813,5 @@
     <link name="left_elbow_extensor">
       <inertial>
-        <mass value="3"/>
+        <mass value="2"/>
         <origin xyz="0.0 0.0 -0.1"/>
         <inertia ixx="0.028125" ixy="0" ixz="0" iyy="0.045" iyz="0" izz="0.028125"/>
@@ -844,5 +844,5 @@
     <link name="left_wrist_rotator">
       <inertial>
-        <mass value="3"/>
+        <mass value="2"/>
         <origin xyz="0.0 0.0 -0.02"/>
         <inertia ixx="0.028125" ixy="0" ixz="0" iyy="0.045" iyz="0" izz="0.028125"/>
@@ -875,5 +875,5 @@
     <link name="left_wrist_extensor">
       <inertial>
-        <mass value="3"/>
+        <mass value="1"/>
         <origin xyz="0.0 0.0 -0.02"/>
         <inertia ixx="0.028125" ixy="0" ixz="0" iyy="0.045" iyz="0" izz="0.028125"/>
@@ -906,5 +906,5 @@
     <link name="left_wrist_adductor">
       <inertial>
-        <mass value="3"/>
+        <mass value="1"/>
         <origin xyz="0.0 0.0 -0.06"/>
         <inertia ixx="0.028125" ixy="0" ixz="0" iyy="0.045" iyz="0" izz="0.028125"/>
@@ -937,5 +937,5 @@
     <link name="neck_rotator">
       <inertial>
-        <mass value="3"/>
+        <mass value="0.5"/>
         <origin xyz="0.0 0.0 0.01"/>
         <inertia ixx="0.0028125" ixy="0" ixz="0" iyy="0.0045" iyz="0" izz="0.0028125"/>
@@ -968,5 +968,5 @@
     <link name="neck_extensor">
       <inertial>
-        <mass value="3"/>
+        <mass value="0.5"/>
         <origin xyz="0.0 0.0 0.01"/>
         <inertia ixx="0.0028125" ixy="0" ixz="0" iyy="0.0045" iyz="0" izz="0.0028125"/>
@@ -999,5 +999,5 @@
     <link name="neck_adductor">
       <inertial>
-        <mass value="3"/>
+        <mass value="0.5"/>
         <origin xyz="0.0 0.0 0.01"/>
         <inertia ixx="0.0028125" ixy="0" ixz="0" iyy="0.0045" iyz="0" izz="0.0028125"/>
@@ -1030,5 +1030,5 @@
     <link name="head">
       <inertial>
-        <mass value="3"/>
+        <mass value="2"/>
         <origin xyz="0.0 0.0 0.11"/>
         <inertia ixx="0.0028125" ixy="0" ixz="0" iyy="0.0045" iyz="0" izz="0.0028125"/>
