Commit message: Fixed indentation.

File: stickbot_lowerleg_3dof/models/stickbot_lowerleg_3dof/xacro/stickbot_lowerleg_3dof_base.xacro (robot description, xacro)
@@ -13,5 +13,5 @@
                 <origin rpy="0 0 0 " xyz="0 0 0.01"/>
                 <geometry name="foot">
-                <box size="0.5 0.3 0.04"/> <!-- NOTE: These dimensions don't match inertial dimensions -->
+                    <box size="0.5 0.3 0.04"/> <!-- NOTE: These dimensions don't match inertial dimensions -->
                 </geometry>
                 <material name="grey">
